File: hw/motherboard/project/HSLF.kicad_sch (KiCad schematic)
At the start: 76 parts, among them J1 JST_01x02_Pin, J2 Conn_01x12_Pin, J3 JST_01x02_Pin, J4 JST_01x02_Pin, J5 IDC_Conn_STLink-V2, J6 USB4940-00-A, J7 XT60-M, Q1 Q_NMOS_DGS, Q2 AO3401A, SW1 SW_Push, SW2 SW_Push, SW3 SW_SPDT, U1 STM32F103C8T6, U2 TPS563201, U3 AMS1117-5.0, U4 VS1838B, U5 A4950E, U6 A4950E, Y1 16MHz

Commit message: schematic revision
Connections:
- net Conn_USBC_D+: now also J6.B6 (DP2)
- net Conn_USBC_D-: now also J6.B7 (DN2)
- net USBC_D+: no longer J6.B6 (DP2)
- net USBC_D-: no longer J6.B7 (DN2)
Changed lines of the file:
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@@
 		(title "HSFL MotherBoard")
 		(date "2026-07-16")
-		(rev "0")
+		(rev "1")
 		(company "Kauê Lucas Nascimento da Silva & Laio")
 	)
@@
 	(wire
 		(pts
-			(xy 320.04 140.97) (xy 330.2 140.97)
-		)
-		(stroke
-			(width 0)
-			(type default)
-		)
-	)
-	(wire
-		(pts
 			(xy 237.49 58.42) (xy 213.36 58.42)
 		)
@@
 	(wire
 		(pts
+			(xy 312.42 133.35) (xy 327.66 133.35)
+		)
+		(stroke
+			(width 0)
+			(type default)
+		)
+	)
+	(wire
+		(pts
 			(xy 363.22 151.13) (xy 363.22 154.94)
 		)
@@
 	(wire
 		(pts
+			(xy 330.2 143.51) (xy 330.2 130.81)
+		)
+		(stroke
+			(width 0)
+			(type default)
+		)
+	)
+	(wire
+		(pts
+			(xy 327.66 140.97) (xy 327.66 133.35)
+		)
+		(stroke
+			(width 0)
+			(type default)
+		)
+	)
+	(wire
+		(pts
 			(xy 262.89 165.1) (xy 270.51 165.1)
 		)
@@
 	(wire
 		(pts
+			(xy 312.42 130.81) (xy 330.2 130.81)
+		)
+		(stroke
+			(width 0)
+			(type default)
+		)
+	)
+	(wire
+		(pts
 			(xy 39.37 49.53) (xy 39.37 54.61)
 		)
@@
 	(wire
 		(pts
+			(xy 320.04 140.97) (xy 327.66 140.97)
+		)
+		(stroke
+			(width 0)
+			(type default)
+		)
+	)
+	(wire
+		(pts
 			(xy 383.54 151.13) (xy 389.89 151.13)
 		)
@@
 		)
 	)
+	(label "Conn_USBC_D-"
+		(at 312.42 130.81 0)
+		(effects
+			(font
+				(size 1.27 1.27)
+			)
+			(justify left bottom)
+		)
+	)
 	(label "LED"
 		(at 251.46 241.3 0)
@@
 		)
 	)
-	(label "USBC_D+"
-		(at 330.2 140.97 180)
-		(effects
-			(font
-				(size 1.27 1.27)
-			)
-			(justify right bottom)
-		)
-	)
 	(label "TX_IR"
 		(at 238.76 140.97 180)
@@
 		)
 	)
-	(label "SWDIO"
-		(at 270.51 165.1 180)
+	(label "Conn_USBC_D+"
+		(at 312.42 133.35 0)
 		(effects
 			(font
 				(size 1.27 1.27)
 			)
-			(justify right bottom)
+			(justify left bottom)
 		)
 	)
-	(label "CC2"
-		(at 321.31 138.43 0)
+	(label "SWDIO"
+		(at 270.51 165.1 180)
 		(effects
 			(font
 				(size 1.27 1.27)
 			)
-			(justify left bottom)
+			(justify right bottom)
 		)
 	)
-	(label "USBC_D-"
-		(at 330.2 143.51 180)
+	(label "CC2"
+		(at 321.31 138.43 0)
 		(effects
 			(font
 				(size 1.27 1.27)
 			)
-			(justify right bottom)
+			(justify left bottom)
 		)
 	)

Commit message: schematic finalized rev 1.1
Parts:
- removed R11: 100, symbol Device:R_Small
- added R22: 100, symbol Device:R
Connections:
- net 5VA: now also R22.2
- net at C18.1, R10.1, U4.3 (Vs): now also R22.1
