File: hw/motherboard/project/HSLF.kicad_pcb (KiCad board)
At the start: 2 copper layers, 120 x 65.1 mm, 76 parts, among them J1 JST_01x02_Pin, J2 Conn_01x12_Pin, J3 JST_01x02_Pin, J4 JST_01x02_Pin, J5 IDC_Conn_STLink-V2, J6 USB4940-00-A, J7 XT30-M, Q1 Q_NMOS_DGS, Q2 AO3401A, SW1 SW_Push, SW2 SW_Push, SW3 SW_SPDT, U1 STM32F103C8T6, U2 TPS563201, U3 AMS1117-5.0, U4 VS1838B, U5 A4950E, U6 A4950E, Y1 16MHz

Commit message: Finalize the V1 MotherBoard PCB
Parts:
- J7: footprint Connector_AMASS:AMASS_XT30UPB-M_1x02_P5.0mm_Vertical -> Connector_AMASS:AMASS_XT30U-M_1x02_P5.0mm_Vertical
- moved R8 46.5 mm to (181.7, 79.7), turned to 180 degrees
- moved C8 7.40 mm to (121.9, 65.2), turned to 0 degrees
- moved R10 6.83 mm to (122.5, 70.7), turned to 180 degrees
- moved R9 2.32 mm to (117.9, 64.4)
- moved TP3 2.14 mm to (115.5, 66.0)
- moved C3 1.80 mm to (119.7, 76.2)
- moved J7 1.68 mm to (192.1, 105.4)
- moved TP1 1.51 mm to (198.1, 106.4)
- moved C19 1.06 mm to (133.2, 67.3), turned to 90 degrees
- moved D1 0.51 mm to (108.5, 63.4)
- moved D4 0.37 mm to (113.6, 63.4)
- moved R22 0.25 mm to (131.1, 72.5)
- moved C4 0.21 mm to (113.5, 80.6)
- moved C18 0.20 mm to (129.1, 72.5)
Routing:
- net MOTOR_ESQ2: track 0.00 -> 210.5 mm, vias 0 -> 4
- net MOTOR_ESQ1: track 0.00 -> 201.3 mm, vias 0 -> 4
- net exaustor: track 0.00 -> 172.2 mm, vias 0 -> 6
- net /SWCLK: track 0.00 -> 149.0 mm, vias 0 -> 5
- net /SWDIO: track 0.00 -> 122.3 mm, vias 0 -> 1
- net /RST: track 11.6 -> 125.2 mm, vias 0 -> 1
- net 5VA: track 80.9 -> 181.1 mm, vias 3 -> 6
- net +3V3: track 176.7 -> 272.0 mm, vias 1 -> 4
- net A0: track 0.00 -> 56.1 mm, vias 0 -> 1
- net A1: track 0.00 -> 53.6 mm, vias 0 -> 1
- net A2: track 0.00 -> 49.9 mm, vias 0 -> 1
- net A3: track 0.00 -> 47.7 mm, vias 0 -> 1
- net A4: track 0.00 -> 45.4 mm, vias 0 -> 1
- net A5: track 0.00 -> 43.8 mm, vias 0 -> 1
- net A6: track 0.00 -> 43.0 mm, vias 0 -> 1
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